File: speaker drivers.sch (KiCad schematic (older format))
At the start: 32 parts, among them CN1 68uFE, CN2 10uFE, CN3 0.1uFC

Commit message: Speaker drivers V1 ready for fabrication
Parts:
- removed LOUT1, ROUT1: BNC, LBHB:BNC_Socket_TYCO-AMP_RevA_Date21Jun2010, symbol BNC
- added OUT1: CONN_01X04, Socket_Strips:Socket_Strip_Straight_1x04, symbol CONN_01X04
- RL1, RL2, RL3, RR1, RR2, RR3: footprint Discret:R3 -> Discret:R7
Connections:
- wire segments 114 -> 112

Commit message: Fixes to speaker driver circuit
* Ensure bypass caps between -12V and GND are correct orientation
* Add notation for all caps indicating size
* Widen drill holes in BUF634
* Ensure cap symbols show orientation when needed
Parts:
- removed DPWR1: CONN_01X03, symbol CONN_01X03
- added DPWR1: CONN_01X02, Socket_Strips:Socket_Strip_Angled_1x02, symbol CONN_01X02
- APWR1: footprint (none) -> Socket_Strips:Socket_Strip_Angled_1x03
- CL1, CL3, CR1, CR3: footprint Discret:C1 -> Capacitors_ThroughHole:Capacitor5x6RM2.5
- RL1, RL2, RL3, RR1, RR2, RR3: footprint Discret:R7 -> Discret:R3
Connections:
- no-connect marks 66 -> 65
Changed lines of the file:
@@
 F 0 "RL2" V 7730 650 40  0000 C CNN
 F 1 "5k" V 7657 651 40  0000 C CNN
-F 2 "Discret:R7" V 7580 650 30  0001 C CNN
+F 2 "Discret:R3" V 7580 650 30  0001 C CNN
 F 3 "" H 7650 650 30  0000 C CNN
 	1    7650 650
@@
 F 0 "RL1" V 6080 650 40  0000 C CNN
 F 1 "5k" V 6007 651 40  0000 C CNN
-F 2 "Discret:R7" V 5930 650 30  0001 C CNN
+F 2 "Discret:R3" V 5930 650 30  0001 C CNN
 F 3 "" H 6000 650 30  0000 C CNN
 	1    6000 650
@@
 F 0 "RL3" V 6430 2525 40  0000 C CNN
 F 1 "100k" V 6357 2526 40  0000 C CNN
-F 2 "Discret:R7" V 6280 2525 30  0001 C CNN
+F 2 "Discret:R3" V 6280 2525 30  0001 C CNN
 F 3 "" H 6350 2525 30  0000 C CNN
 	1    6350 2525
@@
 F 0 "RR2" V 7730 3650 40  0000 C CNN
 F 1 "5k" V 7657 3651 40  0000 C CNN
-F 2 "Discret:R7" V 7580 3650 30  0001 C CNN
+F 2 "Discret:R3" V 7580 3650 30  0001 C CNN
 F 3 "" H 7650 3650 30  0000 C CNN
 	1    7650 3650
@@
 F 0 "RR1" V 6080 3650 40  0000 C CNN
 F 1 "5k" V 6007 3651 40  0000 C CNN
-F 2 "Discret:R7" V 5930 3650 30  0001 C CNN
+F 2 "Discret:R3" V 5930 3650 30  0001 C CNN
 F 3 "" H 6000 3650 30  0000 C CNN
 	1    6000 3650
@@
 F 0 "RR3" V 6430 5525 40  0000 C CNN
 F 1 "100k" V 6357 5526 40  0000 C CNN
-F 2 "Discret:R7" V 6280 5525 30  0001 C CNN
+F 2 "Discret:R3" V 6280 5525 30  0001 C CNN
 F 3 "" H 6350 5525 30  0000 C CNN
 	1    6350 5525
@@
 F 0 "CL1" H 8300 1425 40  0000 L CNN
 F 1 "10uFT" H 8306 1240 40  0000 L CNN
-F 2 "Discret:C1" H 8338 1175 30  0001 C CNN
+F 2 "Capacitors_ThroughHole:Capacitor5x6RM2.5" H 8338 1175 30  0001 C CNN
 F 3 "" H 8300 1325 60  0000 C CNN
 	1    8300 1325
@@
 F 0 "CL3" H 8300 2825 40  0000 L CNN
 F 1 "10uFT" H 8306 2640 40  0000 L CNN
-F 2 "Discret:C1" H 8338 2575 30  0001 C CNN
+F 2 "Capacitors_ThroughHole:Capacitor5x6RM2.5" H 8338 2575 30  0001 C CNN
 F 3 "" H 8300 2725 60  0000 C CNN
 	1    8300 2725
-	-1   0    0    -1
+	1    0    0    1
 $EndComp
 $Comp
@@
 F 0 "CR1" H 8300 4425 40  0000 L CNN
 F 1 "10uFT" H 8306 4240 40  0000 L CNN
-F 2 "Discret:C1" H 8338 4175 30  0001 C CNN
+F 2 "Capacitors_ThroughHole:Capacitor5x6RM2.5" H 8338 4175 30  0001 C CNN
 F 3 "" H 8300 4325 60  0000 C CNN
 	1    8300 4325
@@
 F 0 "CR3" H 8300 5825 40  0000 L CNN
 F 1 "10uFT" H 8306 5640 40  0000 L CNN
-F 2 "Discret:C1" H 8338 5575 30  0001 C CNN
+F 2 "Capacitors_ThroughHole:Capacitor5x6RM2.5" H 8338 5575 30  0001 C CNN
 F 3 "" H 8300 5725 60  0000 C CNN
 	1    8300 5725
-	-1   0    0    -1
+	1    0    0    1
 $EndComp
 $Comp
@@
 F 0 "APWR1" H 4900 5900 50  0000 C CNN
 F 1 "CONN_01X03" V 5000 5700 50  0000 C CNN
-F 2 "" H 4900 5700 60  0000 C CNN
+F 2 "Socket_Strips:Socket_Strip_Angled_1x03" H 4900 5700 60  0001 C CNN
 F 3 "" H 4900 5700 60  0000 C CNN
 	1    4900 5700
 	0    -1   -1   0
 $EndComp
-$Comp
-L CONN_01X03 DPWR1
-U 1 1 54341684
-P 5500 5700
-F 0 "DPWR1" H 5500 5900 50  0000 C CNN
-F 1 "CONN_01X03" V 5600 5700 50  0000 C CNN
-F 2 "" H 5500 5700 60  0000 C CNN
-F 3 "" H 5500 5700 60  0000 C CNN
-	1    5500 5700
-	0    -1   -1   0
-$EndComp
 Wire Wire Line
 	2050 5575 2050 5850
@@
 Wire Wire Line
 	5600 6150 5600 5900
-NoConn ~ 5400 5900
+$Comp
+L CONN_01X02 DPWR1
+U 1 1 5434245A
+P 5550 5700
+F 0 "DPWR1" H 5550 5850 50  0000 C CNN
+F 1 "CONN_01X02" V 5650 5700 50  0000 C CNN
+F 2 "Socket_Strips:Socket_Strip_Angled_1x02" H 5550 5700 60  0001 C CNN
+F 3 "" H 5550 5700 60  0000 C CNN
+	1    5550 5700
+	0    -1   -1   0
+$EndComp
 $EndSCHEMATC

Commit message: Connect P0.0 to PFI0 ... PFI2 in speaker drivers circuit
Connections:
- wire segments 112 -> 117
- no-connect marks 65 -> 61
Changed lines of the file:
@@
 LIBS:lbhb
 LIBS:speaker drivers-cache
-EELAYER 24 0
+EELAYER 25 0
 EELAYER END
 $Descr A4 11693 8268
@@
 NoConn ~ 2925 2975
 NoConn ~ 2925 3075
-NoConn ~ 1075 1475
 NoConn ~ 1075 1675
-NoConn ~ 1075 2375
-NoConn ~ 1075 2475
-NoConn ~ 1075 2575
 NoConn ~ 1075 2675
 NoConn ~ 1075 2775
@@
 	0    -1   -1   0
 $EndComp
+Wire Wire Line
+	1075 2375 950  2375
+Wire Wire Line
+	950  1475 950  2575
+Wire Wire Line
+	950  2475 1075 2475
+Connection ~ 950  2375
+Wire Wire Line
+	950  2575 1075 2575
+Connection ~ 950  2475
+Wire Wire Line
+	950  1475 1075 1475
 $EndSCHEMATC

Commit message: Commit before modifying speaker driver schematic
Parts:
- removed CG1: 150uFE, Capacitors_ThroughHole:Capacitor5x6RM2.5, symbol CP2
- removed CN1, CP1: 68uFE, Capacitors_ThroughHole:Capacitor5x6RM2.5, symbol CP2
- removed DPWR1: CONN_01X02, Socket_Strips:Socket_Strip_Angled_1x02, symbol CONN_01X02
- removed H1: NI_header, LBHB:2x2x18, symbol NI_header
- removed OUT1: CONN_01X04, Socket_Strips:Socket_Strip_Straight_1x04, symbol CONN_01X04
- added COMM1: CONN_01X05, Socket_Strips:Socket_Strip_Straight_1x05, symbol CONN_01X05
- added OUTL1, OUTR1: BNC, LBHB:BNC_Socket_TYCO-AMP_RevA_Date21Jun2010, symbol BNC
- added SIG1: CONN_01X03, symbol CONN_01X03
- APWR1: footprint Socket_Strips:Socket_Strip_Angled_1x03 -> Socket_Strips:Socket_Strip_Straight_1x03
- RL1, RL2, RL3, RR1, RR2, RR3: footprint Discret:R3 -> Discret:R5
Connections:
- wire segments 117 -> 103
- no-connect marks 61 -> 1
Other:
- note removed: "CS/SCLK/SDI must be on port 0 for M-series"

Commit message: ENH: Working draft of speaker drivers v2
Parts:
- removed APWR1: CONN_01X03, Socket_Strips:Socket_Strip_Straight_1x03, symbol CONN_01X03
- removed CG3: 0.1uFC, Discret:C1, symbol C
- removed CL3, CR3: 10uFT, Capacitors_ThroughHole:Capacitor5x6RM2.5, symbol CP2
- removed COMM1: CONN_01X05, Socket_Strips:Socket_Strip_Straight_1x05, symbol CONN_01X05
- removed CTL1: PGA2310, Sockets_DIP:DIP-16__300_ELL, symbol PGA2310
- removed OUTL1, OUTR1: BNC, LBHB:BNC_Socket_TYCO-AMP_RevA_Date21Jun2010, symbol BNC
- removed SIG1: CONN_01X03, symbol CONN_01X03
- added BUFL2, BUFR2: BUF634, LBHB:BUF634, symbol BUF634
- added CL2, CR2: 10uFT, Capacitors_ThroughHole:Capacitor5x6RM2.5, symbol CP2
- added CL3, CR3: 2uF, Discret:C1, symbol C
- added Cvr1: 0.33uF, Discret:C1, symbol C
- added Cvr2: 0.1uF, Discret:C1, symbol C
- added LL1, LR1: 100uH, symbol INDUCTOR
- added PWR1: 4P_miniDIN_PWR, symbol 4P_miniDIN_PWR
- added RL4, RR4: 22, Discret:R5, symbol R
- added RS1: 100k, Discret:R5, symbol R
- added SER1: 8P_miniDIN, symbol 8P_miniDIN
- added SIGIN1, SIGOUT1: 4P_miniDIN, symbol 4P_miniDIN
- added VCTL1: PGA2310, symbol PGA2310
- added VREG1: 78L05, symbol 78L05
- renumbered C3 to C2
Connections:
- net labels removed: +5V
- wire segments 103 -> 139
- no-connect marks 1 -> 3
Other:
- moved on the sheet: BUFR1, C1, C2, CG2, CLin1, CN2, CN3, CP2, CP3, CR1, CRin1, OPA1A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

Commit message: Commit before major revisions
Parts:
- added CL5, CL6, CR5, CR6: 0.1uF, Discret:C1, symbol C
- RL1, RR1: value 5k -> 100k
Connections:
- net +12V: now also CL6.1, CR6.1
- net -12V: now also CL5.1, CR5.1
- net AGND: now also PWR1.C, SIGIN1.C, SIGOUT1.C, CL5.2, CL6.2, CR5.2, CR6.2
- net DGND: now also RS1.1, SER1.C
- net at CG2.1, Cvr2.2, VCTL1.4 (VD+)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: no longer RS1.1

Commit message: WIP: Preliminary commit before splitting boards
Parts:
- removed CG2: 10uFE, Capacitors_ThroughHole:Capacitor5x6RM2.5, symbol CP2
- removed Cvr1: 0.33uF, Discret:C1, symbol C
- removed Cvr2: 0.1uF, Discret:C1, symbol C
- removed PWR1: 4P_miniDIN_PWR, symbol 4P_miniDIN_PWR
- removed RS1: 100k, Discret:R5, symbol R
- removed SER1: 8P_miniDIN, symbol 8P_miniDIN
- removed SIGIN1, SIGOUT1: 4P_miniDIN, symbol 4P_miniDIN
- removed VCTL1: PGA2310, symbol PGA2310
- removed VREG1: 78L05, symbol 78L05
- added BNCLin1, BNCRin1: BNC, Socket_Strips:Socket_Strip_Straight_1x02, symbol BNC
- added JL1, JR1: JUMPER, Socket_Strips:Socket_Strip_Straight_1x02, symbol JUMPER
- added JL2, JR2: JUMPER3, Socket_Strips:Socket_Strip_Straight_1x03, symbol JUMPER3
- added Lout1, Rout1: CONN_01X02, Socket_Strips:Socket_Strip_Straight_1x02, symbol CONN_01X02
- added PWR1: CONN_01X03, Socket_Strips:Socket_Strip_Straight_1x03, symbol CONN_01X03
- C1, C2, CL5, CL6, CN3, CP3, CR5, CR6: footprint Discret:C1 -> LBHB:capacitor-2.5x5mm-L_2.5mm
- CL1, CL2, CN2, CP2, CR1, CR2: footprint Capacitors_ThroughHole:Capacitor5x6RM2.5 -> LBHB:capacitor-D_4mm-L_2.4mm
- CL3, CLin1, CR3, CRin1: footprint Discret:C1 -> LBHB:capacitor-D_5mm-L_2mm
- LL1, LR1: footprint (none) -> LBHB:inductor-12mm
- OPA1: footprint Sockets_DIP:DIP-8__300_ELL -> LBHB:DIP-8
- RL1, RL3, RR1, RR3: footprint Discret:R5 -> LBHB:resistor-6x2.3mm
- RL2, RR2: footprint Discret:R5 -> LBHB:resistor-4x2mm
- RL4, RR4: footprint Discret:R5 -> LBHB:resistor-13x4mm
Connections:
- net +12V: now also OPA1.8 (V+), PWR1.3 (P3); no longer OPA1.8 (V+)
- net -12V: now also OPA1.4 (V-), PWR1.1 (P1); no longer OPA1.4 (V-)
- net AGND: now also JL1.1, JR1.1, Lout1.2 (P2), PWR1.2 (P2), Rout1.2 (P2); no longer RL1.2, RR1.2
- net at BUFL1.2, BUFL2.2: now also OPA1.7; no longer OPA1.1
- net at RL1.1, RL2.2: now also OPA1.6 (-), JL2.2; no longer OPA1.2 (-)
- net at OPA1.3 (+): now also CRin1.1, RR3.2; no longer RL3.2
- net at CLin1.1: now also OPA1.5 (+), RL3.2
- net at CLin1.2: now also BNCLin1.1 (In)
- net at RR1.1, RR2.2: now also OPA1.2 (-), JR2.2; no longer OPA1.6 (-)
- net at CRin1.2: now also BNCRin1.1 (In)
- net at BUFR1.2, BUFR2.2: now also OPA1.1; no longer OPA1.7
- net at CR3.2, LR1.2: now also Rout1.1 (P1)
- net at CL3.2, LL1.2: now also Lout1.1 (P1)
- new net: JL1.2, JL2.3, RL1.2
- new net: BNCLin1.2 (Ext), JL2.1
- new net: JR1.2, JR2.3, RR1.2
- new net: BNCRin1.2 (Ext), JR2.1
- no-connect marks 3 -> 0
Other:
- moved on the sheet: BUFL1, BUFL2, BUFR1, BUFR2, C1, C2, CL1, CL2, CL3, CL5, CL6, CLin1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

Commit message: WIP: Test of new circuit for speaker drivers
Note that this circuit does not work and should not be used for
production.
Parts:
- removed BNCRin1: BNC, Socket_Strips:Socket_Strip_Straight_1x02, symbol BNC
- removed BUFR1, BUFR2: BUF634, LBHB:BUF634, symbol BUF634
- removed C1, C2, CN3, CP3: 0.1uFC, LBHB:capacitor-2.5x5mm-L_2.5mm, symbol C
- removed CL3, CR3: 2uF, LBHB:capacitor-D_5mm-L_2mm, symbol C
- removed CN2, CP2: 10uFE, LBHB:capacitor-D_4mm-L_2.4mm, symbol CP2
- removed CR1, CR2: 10uFT, LBHB:capacitor-D_4mm-L_2.4mm, symbol CP2
- removed CR5, CR6: 0.1uF, LBHB:capacitor-2.5x5mm-L_2.5mm, symbol C
- removed CRin1: 1uF, LBHB:capacitor-D_5mm-L_2mm, symbol C
- removed JL1, JR1: JUMPER, Socket_Strips:Socket_Strip_Straight_1x02, symbol JUMPER
- removed JL2, JR2: JUMPER3, Socket_Strips:Socket_Strip_Straight_1x03, symbol JUMPER3
- removed LL1, LR1: 100uH, LBHB:inductor-12mm, symbol INDUCTOR
- removed Lout1, Rout1: CONN_01X02, Socket_Strips:Socket_Strip_Straight_1x02, symbol CONN_01X02
- removed OPA1: OPA2134, LBHB:DIP-8, symbol OPA2134
- removed RL2, RR2: 5k, LBHB:resistor-4x2mm, symbol R
- removed RL3, RR1, RR3: 100k, LBHB:resistor-6x2.3mm, symbol R
- removed RL4, RR4: 22, LBHB:resistor-13x4mm, symbol R
- added C10, C3, C4: 0.1uF, LBHB:capacitor-2x4mm-L_2.5mm, symbol C-RESCUE-speaker_drivers
- added C2: 1.2nF, Capacitors_ThroughHole:C_Disc_D6_P5, symbol C-RESCUE-speaker_drivers
- added C9: 68nF, Capacitors_ThroughHole:C_Disc_D6_P5, symbol C-RESCUE-speaker_drivers
- added O1: OPA134, Housings_DIP:DIP-8_W7.62mm_LongPads, symbol OPA134
- added P1: CONN_01X02, Socket_Strips:Socket_Strip_Straight_1x02, symbol CONN_01X02
- added R2, R5: 1k, Discret:R3-5, symbol R-RESCUE-speaker_drivers
- added R3: 49.9, Discret:R3, symbol R-RESCUE-speaker_drivers
- added R4: 8.2, Discret:R4-5, symbol R-RESCUE-speaker_drivers
- C1: renamed from CLin1; value 1uF -> 33nF; footprint LBHB:capacitor-D_5mm-L_2mm -> Capacitors_ThroughHole:C_Disc_D6_P5; symbol C -> C-RESCUE-speaker_drivers
- CL1, CL2: value 10uFT -> 10uF
- CL5, CL6: footprint LBHB:capacitor-2.5x5mm-L_2.5mm -> LBHB:capacitor-2x4mm-L_2.5mm; symbol C -> C-RESCUE-speaker_drivers
- R1: renamed from RL1; value 100k -> 10k; footprint LBHB:resistor-6x2.3mm -> Discret:R3-5; symbol R -> R-RESCUE-speaker_drivers
- renumbered BUFL1 to B1, BUFL2 to B2, BNCLin1 to V1
Connections:
- net +12V: now also C4.2, O1.4 (V-)
- net -12V: now also C3.2, O1.7 (V+)
- net AGND: now also V1.2 (Ext), C10.1, C3.1, C4.1, C9.1, P1.2 (P2), R3.1, R5.1
- net at B1.4, B2.4: now also C2.1, R4.2
- net at R1.1: now also C2.2, O1.2 (-), R2.2
- net at R1.2: now also C1.1
- net at C1.2, V1.1 (In): now also R3.2
- net at B1.2, B2.2: now also O1.6
- new net: C10.2, O1.3 (+), R5.2
- new net: C9.2, P1.1 (P1), R2.1, R4.1
Other:
- note removed: "Design notes:\n* NI M-series boards have an analog range of -10 to 10V, so we only need \nunity gain. BUF634 is used to provide high-current, OPA2134 is used to \nstablize voltage output of BUF634.\n* Bypass capacitors are speced as ceramic (C), metal film electrolytic (E) or tantalum (T)\n* BUF634 should have wide-bandwidth mode enabled by shorting pin 1 to V-\nto ensure stable operation when dr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"
- moved on the sheet: B1, B2, C1, CL1, CL2, CL5, CL6, PWR1, R1, V1
